File: Breakout Board/eeArm_Breakout.brd (EAGLE design)
At the start: 29.2 x 30.5 mm, 22 parts, among them X1 ESP8266

Commit message: Started with labels
Parts:
- moved R2 0.76 mm to (21.7, 12.7)
Other:
- board text added: "+"
- board text added: "+3V3"
- board text added: "-"
- board text added: "0"
- board text added: "12"
- board text added: "13"
- board text added: "14"
- board text added: "15"
- board text added: "16"
- board text added: "2"
- board text added: "4"
- board text added: "5"
- board text added: "ADC"
- board text added: "EN"
- board text added: "GND"
- board text added: "RST"
- board text added: "RX"
- board text added: "TX"
- board text added: "VIN"
