File: Breakout Board/eeArm_Breakout.brd (EAGLE design)
At the start: 29.2 x 30.5 mm, 23 parts, among them X1 ESP8266

Commit message: Go time
Parts:
- removed R5: 4K7, resistor:R0805
- added R1: 4K7, resistor:R0805
- moved R2 10.6 mm to (11.4, 10.2)
- moved R4 10.6 mm to (21.7, 10.2)
- moved R3 9.86 mm to (18.4, 10.2), turned to 270 degrees
- moved D1 2.79 mm to (7.11, 3.81)
- moved C1 2.67 mm to (6.35, 2.03)
- moved E$1 2.54 mm to (24.1, 24.1)
- moved BASE 2.54 mm to (14.0, 6.60)
- moved BODY 2.54 mm to (17.1, 6.60)
- moved CLAW 2.54 mm to (23.5, 6.60)
- moved JP2 2.54 mm to (27.3, 7.62)
- moved JP3 2.54 mm to (1.91, 5.08)
- moved NECK 2.54 mm to (20.3, 6.60)
- moved POWER 2.54 mm to (10.8, 4.06)
- moved RESET 2.54 mm to (6.99, 4.45)
- moved U$8 2.54 mm to (1.91, 1.91)
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Connections:
- net +3V3: now also R1.1, R2.1, R3.2; no longer R3.1, R4.1, R5.2
- net CH_PD: now also R1.2; no longer R3.2
- net DTR: now also R3.1; no longer R5.1
- net GND: now also R4.1; no longer R2.1
- net GPIO15: now also R4.2; no longer R2.2
- net RESET: now also R2.2; no longer R4.2
Routing:
- net GND: track 0.00 -> 7.60 mm
- net BASE: track 32.7 -> 33.5 mm
- net VBATT: track 25.4 -> 26.1 mm
Other:
- board text added: "3V3"
- board text added: "BASE"
- board text added: "BODY"
- board text added: "C1"
- board text added: "C2"
- board text added: "CLAW"
- board text added: "D1"
- board text added: "NECK"
- board text added: "PWR"
- board text added: "R1"
- board text added: "R2"
- board text added: "R3"
- board text added: "R4"
- board text added: "VREG1"
- board text removed: "+3V3"
