File: Breakout Board/eeArm_Breakout_Panelized.brd (EAGLE design)
At the start: 29.2 x 30.5 mm, 23 parts, among them X1 ESP8266

Commit message: Ready for panelising
Parts:
- added BASE1, BODY1, CLAW1, NECK1: (no value), SparkFun-Connectors:1X03_LOCK
- added C3: 100n, resistor:C0805
- added C4: 10u, resistor:C0805
- added D2: MBR120, microbuilder:SOD-123
- added E$3: (no value), Gwa's Parts:MAKERSPACE_LOGO
- added E$4: (no value), Gwaja-logo:GWAJA-LOGO-PLACE
- added JP1: J1, SparkFun-Connectors:1X08_LOCK
- added JP4: (no value), SparkFun-Connectors:1X09_LOCK
- added POWER1: (no value), SparkFun-Connectors:1X02_LOCK
- added R1, R6, R7, R8: 4K7, resistor:R0805
- added RESET1: SW_TACT_2P-3X6, Gwa's Parts:SW_TACT_3X6
- added U$1, U$2, U$3, U$4: MOUNTINGHOLE2.0, microbuilder:MOUNTINGHOLE_2.0_PLATED
- added VREG2: LD1117, dp_devices:SOT-223
- added X2: ESP8266, Gwa's Parts:ESP-12-NOPLACE
- moved E$1 2.54 mm to (24.1, 24.1)
- moved BASE 2.54 mm to (14.0, 6.60)
- moved BODY 2.54 mm to (17.1, 6.60)
- moved C1 2.54 mm to (6.35, 2.16)
- moved CLAW 2.54 mm to (23.5, 6.60)
- moved D1 2.54 mm to (7.11, 4.06)
- moved JP2 2.54 mm to (27.3, 7.62)
- moved JP3 2.54 mm to (1.91, 5.08)
- moved NECK 2.54 mm to (20.3, 6.60)
- moved POWER 2.54 mm to (10.8, 4.06)
- moved RESET 2.54 mm to (6.99, 4.45)
- moved U$8 2.54 mm to (1.91, 1.91)
- moved U$9 2.54 mm to (27.3, 1.91)
- moved C2 2.54 mm to (12.6, 9.27)
- moved E$2 2.54 mm to (24.9, 9.91)
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Connections:
- new net +3V1: C4.1, JP4.2, R6.1, R7.1, R8.2, VREG2.2, X2.8
- new net ADC1: JP4.8, X2.2
- new net BASE1: BASE1.1, JP4.3, X2.7
- new net BODY1: BODY1.1, JP4.4, X2.6
- new net CH_PD1: JP4.7, R6.2, X2.3
- new net CLAW1: CLAW1.1, JP4.6, X2.4
- new net DTR1: JP1.4, R8.1, X2.12
- new net GND1: BASE1.3, BODY1.3, C3.2, C4.2, CLAW1.3, JP1.1, NECK1.3, POWER1.2, R1.1, RESET1.1, VREG2.1, X2.9
- new net GPIO1: JP1.5, X2.13
- new net GPIO3: JP1.3, X2.11
- new net GPIO6: JP1.6, X2.14
- new net GPIO7: JP1.2, R1.2, X2.10
- new net NECK1: JP4.5, NECK1.1, X2.5
- new net RESET1: JP4.9, R7.2, RESET1.2, X2.1
- new net RX1: JP1.7, X2.15
- new net TX1: JP1.8, X2.16
- new net VBATT1: BASE1.2, BODY1.2, CLAW1.2, D2.A, JP4.1, NECK1.2, POWER1.1
- new net VIN1: C3.1, D2.C, VREG2.3
Routing:
- net CLAW1: track 0.00 -> 36.2 mm
- net RESET1: track 0.00 -> 36.2 mm
- net +3V1: track 0.00 -> 35.5 mm, vias 0 -> 1
- net NECK1: track 0.00 -> 34.3 mm
- net BASE1: track 0.00 -> 32.7 mm
- net BODY1: track 0.00 -> 31.4 mm
- net VBATT1: track 0.00 -> 25.4 mm, vias 0 -> 1
- net CH_PD1: track 0.00 -> 22.1 mm
- net DTR1: track 0.00 -> 18.1 mm
- net GPIO7: track 0.00 -> 15.9 mm
- net GPIO3: track 0.00 -> 7.35 mm
- net ADC1: track 0.00 -> 6.52 mm
- net GPIO6: track 0.00 -> 6.49 mm
- net GPIO1: track 0.00 -> 6.46 mm
- net TX1: track 0.00 -> 6.04 mm
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- added copper zone on layer 1, net GND1
- added copper zone on layer 16, net GND1
Other:
- board size 29.2 x 30.5 mm -> 341.8 x 198 mm
